Commit message: Add files via upload

File: urdf/sr5_description.urdf (robot description, URDF)
Before this commit: robot sr5, 12 links, 11 joints
Links:
- removed link base_footprint
- added link link7, mass 0.038745; collision mesh filename=package://sr5_description/meshes/link7.STL; visual mesh filename=package://sr5_description/meshes/link7.STL
- link base_link: mass 1.8568 -> 27.667
- link link1: mass 1.3178 -> 4.3511
- link link2: mass 2.6176 -> 1.3178
- link link3: mass 1.3019 -> 2.6176
- link link4: mass 0.67706 -> 1.3019
- link link5: mass 0.5365 -> 0.67706
- link link6: mass 0.038745 -> 0.5365
Joints:
- removed joint base_footprint_to_base_link
- added joint joint7: type revolute, parent link6, child link7, origin xyz=0 -0.03207 0.0855 rpy=0 0 0, axis 0 0 -1, limit lower=-3.141 upper=3.141 effort=100000 velocity=100
- joint hand_joint: parent link6 -> link7
- joint joint1: axis 0 0 1 -> 0 1 0; limit lower=-3.141 upper=3.141 effort=1000 velocity=6.282 -> lower=-0.5 upper=0.5 effort=100000 velocity=100; origin xyz=0 0 0.03 rpy=0 0 0 -> xyz=0 0 0.075 rpy=0 0 0; type revolute -> prismatic
- joint joint2: axis 0 1 0 -> 0 0 1; limit lower=-2.141 upper=2.141 effort=1000 velocity=6.282 -> lower=-3.141 upper=3.141 effort=1000000 velocity=1000; origin xyz=0 0.045 0.1 rpy=0 0 0 -> xyz=0 0 0.03 rpy=0 0 0
- joint joint3: limit lower=-2.8 upper=2.8 effort=1000 velocity=6.282 -> lower=-2.8 upper=2.8 effort=100000 velocity=100; origin xyz=0 0 0.39975 rpy=0 0 0 -> xyz=0 0.045 0.1 rpy=0 0 0
- joint joint4: axis 0 0 1 -> 0 1 0; limit lower=-3.141 upper=3.141 effort=1000 velocity=6.282 -> lower=-2.7 upper=2.7 effort=100000 velocity=1000; origin xyz=0 -0.045 0.098 rpy=0 0 0 -> xyz=0 0 0.39975 rpy=0 0 0
- joint joint5: axis 0 1 0 -> 0 0 1; limit lower=-3.141 upper=3.141 effort=1000 velocity=6.282 -> lower=-3.141 upper=3.141 effort=100000 velocity=100; origin xyz=0 0.032068 0.30175 rpy=0 0 0 -> xyz=0 -0.045 0.098 rpy=0 0 0
- joint joint6: axis 0 0 1 -> 0 1 0; limit lower=-3.141 upper=3.141 effort=1000 velocity=6.282 -> lower=-3.141 upper=3.141 effort=1000000 velocity=100; origin xyz=0 -0.03207 0.0855 rpy=0 0 0 -> xyz=0 0.032068 0.30175 rpy=0 0 0
- joint left_finger_joint: axis 0 1 0 -> 0 0 0; limit lower=-0.01 upper=0 effort=1000 velocity=1 -> lower=-0.01 upper=0 effort=100000 velocity=100; type prismatic -> fixed
- joint right_finger_joint: axis 0 1 0 -> 0 0 0; limit lower=0 upper=0.01 effort=1000 velocity=1 -> lower=0 upper=0.01 effort=100000 velocity=100; type prismatic -> fixed
- joint virtual_joint: child base_footprint -> base_link

Commit message: Update sr5_description.urdf

File: urdf/sr5_description.urdf (robot description, URDF)
Before this commit: robot sr5_description, 12 links, 11 joints
Links:
- removed link world
Joints:
- removed joint virtual_joint
